Commit message: track.dae

File: vehicle/track_vehicle_launch/track_vehicle_description/urdf/vehicle.xacro (robot description, xacro)
@@ -8,5 +8,5 @@
       <origin xyz="${vehicle_info['/**']['ros__parameters']['wheel_base']/2.0} 0 0" rpy="${pi/2.0} 0 ${pi}"/>
       <geometry>
-        <mesh filename="package://sample_vehicle_description/mesh/lexus.dae" scale="1 1 1"/>
+        <mesh filename="package://sample_vehicle_description/mesh/track.dae" scale="1 1 1"/>
       </geometry>
     </visual>
